Commit message: Add files via upload

File: src/my_robot_description/urdf/emiliobot.urdf.xacro (robot description, xacro)
@@ -1,4 +1,4 @@
 <?xml version="1.0"?>
-<robot name="my_robot" xmlns:xacro="http://www.ros.org/wiki/xacro">
+<robot name="emiliobot" xmlns:xacro="http://www.ros.org/wiki/xacro">
     <xacro:include filename="common_properties.xacro" />
     <xacro:include filename="mobile_base_gazebo.xacro" />
@@ -13,4 +13,10 @@
     <material name="grey">
         <color rgba="0.5 0.5 0.5 1" />
+    </material>
+    <material name="red">
+        <color rgba="0.5 0 0 1" />
+    </material>
+    <material name="black">
+        <color rgba="0 0 0 1" />
     </material>
     <link name="base_footprint" />
@@ -29,5 +35,5 @@
             </geometry>
             <origin xyz="0 0 ${base_height / 2.0}" rpy="0 0 0" />
-            <material name="blue" />
+            <material name="red" />
         </visual>
         <collision>
@@ -39,4 +45,9 @@
         <xacro:box_inertia m="5.0" x="${base_length}" y="${base_width}" z="${base_height}" o_xyz="0 0 ${base_height / 2.0}" o_rpy="0 0 0" />
     </link>
+    <joint name="base_joint" type="fixed">
+        <parent link="base_footprint" />
+        <child link="base_link" />
+        <origin xyz="0 0 ${wheel_radius}" rpy="0 0 0" />
+    </joint>
     <!--
      _____  _____ _____ _    _ _______  __          ___    _ ______ ______ _
@@ -53,5 +64,5 @@
             </geometry>
             <origin xyz="0 0 0" rpy="${pi / 2.0} 0 0" />
-            <material name="grey" />
+            <material name="black" />
         </visual>
         <collision>
@@ -63,4 +74,10 @@
         <xacro:cylinder_inertia m="1.0" r="${wheel_radius}" l="${wheel_length}" o_xyz="0 0 0" o_rpy="${pi / 2.0} 0 0" />
     </link>
+    <joint name="base_right_wheel_joint" type="continuous">
+        <parent link="base_link" />
+        <child link="right_wheel_link" />
+        <origin xyz="${-base_length / 4.0} -0.225 0" rpy="0 0 0" />
+        <axis xyz="0 1 0" />
+    </joint>
     <!--
      _      ______ ______ _______  __          ___    _ ______ ______ _
@@ -77,5 +94,5 @@
             </geometry>
             <origin xyz="0 0 0" rpy="${pi / 2.0} 0 0" />
-            <material name="grey" />
+            <material name="black" />
         </visual>
         <collision>
@@ -87,4 +104,41 @@
         <xacro:cylinder_inertia m="1.0" r="${wheel_radius}" l="${wheel_length}" o_xyz="0 0 0" o_rpy="${pi / 2.0} 0 0" />
     </link>
+    <joint name="base_left_wheel_joint" type="continuous">
+        <parent link="base_link" />
+        <child link="left_wheel_link" />
+        <origin xyz="${-base_length / 4.0} 0.225 0" rpy="0 0 0" />
+        <axis xyz="0 1 0" />
+    </joint>
+    <!--
+      _______ ____  _____   __          ___    _ ______ ______ _
+     |__   __/ __ \|  __ \  \ \        / / |  | |  ____|  ____| |
+        | | | |  | | |__) |  \ \  /\  / /| |__| | |__  | |__  | |
+        | | | |  | |  ___/    \ \/  \/ / |  __  |  __| |  __| | |
+        | | | |__| | |         \  /\  /  | |  | | |____| |____| |____
+        |_|  \____/|_|          \/  \/   |_|  |_|______|______|______|
+    -->
+    <link name="top_wheel_link">
+        <visual>
+            <geometry>
+                <cylinder radius="${wheel_radius}" length="${wheel_length}" />
+            </geometry>
+            <origin xyz="0 0 0" rpy="${pi / 2.0} 0 0" />
+            <material name="black" />
+        </visual>
+        <collision>
+            <geometry>
+                <sphere radius="${wheel_radius}" />
+            </geometry>
+            <origin xyz="0 0 0" rpy="0 0 0" />
+        </collision>
+        <xacro:cylinder_inertia m="1.0" r="${wheel_radius}" l="${wheel_length}" o_xyz="0 0 0" o_rpy="${pi / 2.0} 0 0" />
+    </link>
+    <joint name="base_top_wheel_joint" type="continuous">
+        <parent link="base_link" />
+        <child link="top_wheel_link" />
+        <origin xyz="0 0 ${base_height
+        }" rpy="0 0 0" />
+        <axis xyz="0 1 0" />
+    </joint>
     <!--
       _____           _____ _______ ______ _____   __          ___    _ ______ ______ _
@@ -101,5 +155,5 @@
             </geometry>
             <origin xyz="0 0 0" rpy="0 0 0" />
-            <material name="grey" />
+            <material name="black" />
         </visual>
         <collision>
@@ -111,21 +165,4 @@
         <xacro:sphere_inertia m="0.5" r="${wheel_radius / 2.0}" o_xyz="0 0 0" o_rpy="0 0 0" />
     </link>
-    <joint name="base_joint" type="fixed">
-        <parent link="base_footprint" />
-        <child link="base_link" />
-        <origin xyz="0 0 ${wheel_radius}" rpy="0 0 0" />
-    </joint>
-    <joint name="base_right_wheel_joint" type="continuous">
-        <parent link="base_link" />
-        <child link="right_wheel_link" />
-        <origin xyz="${-base_length / 4.0} -0.225 0" rpy="0 0 0" />
-        <axis xyz="0 1 0" />
-    </joint>
-    <joint name="base_left_wheel_joint" type="continuous">
-        <parent link="base_link" />
-        <child link="left_wheel_link" />
-        <origin xyz="${-base_length /4.0} 0.225 0" rpy="0 0 0" />
-        <axis xyz="0 1 0" />
-    </joint>
     <joint name="base_caster_wheel_joint" type="fixed">
         <parent link="base_link" />

Commit message: Add files via upload

File: src/my_robot_description/urdf/emiliobot.urdf.xacro (robot description, xacro)
@@ -149,4 +149,5 @@
      \_____/_/    \_\_____/   |_|  |______|_|  \_\     \/  \/   |_|  |_|______|______|______|
     -->
+    <!-- Caster wheel link -->
     <link name="caster_wheel_link">
         <visual>
@@ -163,5 +164,12 @@
             <origin xyz="0 0 0" rpy="0 0 0" />
         </collision>
-        <xacro:sphere_inertia m="0.5" r="${wheel_radius / 2.0}" o_xyz="0 0 0" o_rpy="0 0 0" />
+        <inertial>
+            <origin xyz="0 0 0" rpy="0 0 0" />
+            <mass value="0.5" />
+            <inertia
+                ixx="0.001" ixy="0.0" ixz="0.0"
+                iyy="0.001" iyz="0.0"
+                izz="0.001" />
+        </inertial>
     </link>
     <joint name="base_caster_wheel_joint" type="fixed">
@@ -170,3 +178,53 @@
         <origin xyz="${base_length / 3.0} 0 -0.05" rpy="0 0 0" />
     </joint>
+    <!-- ==========================
+         FPV CAMERA FOR EMILIOBOT
+         ========================== -->
+    <link name="camera_link">
+        <visual>
+            <geometry>
+                <box size="0.05 0.05 0.05" />
+            </geometry>
+            <origin xyz="0 0 0" rpy="0 0 0" />
+            <material name="black" />
+        </visual>
+        <collision>
+            <geometry>
+                <box size="0.05 0.05 0.05" />
+            </geometry>
+            <origin xyz="0 0 0" rpy="0 0 0" />
+        </collision>
+        <inertial>
+            <origin xyz="0 0 0" rpy="0 0 0" />
+            <mass value="0.1" />
+            <inertia
+                ixx="0.001" ixy="0.0" ixz="0.0"
+                iyy="0.001" iyz="0.0"
+                izz="0.001" />
+        </inertial>
+    </link>
+    <joint name="camera_joint" type="fixed">
+        <parent link="base_link" />
+        <child link="camera_link" />
+        <origin xyz="0 0 ${base_height + 0.1}" rpy="0 0 0" />
+    </joint>
+    <gazebo reference="camera_link">
+        <sensor name="front_camera" type="camera">
+            <always_on>1</always_on>
+            <update_rate>30</update_rate>
+            <visualize>true</visualize>
+            <camera>
+                <horizontal_fov>1.047</horizontal_fov>
+                <image>
+                    <width>640</width>
+                    <height>480</height>
+                    <format>R8G8B8</format>
+                </image>
+                <clip>
+                    <near>0.1</near>
+                    <far>100.0</far>
+                </clip>
+            </camera>
+        </sensor>
+    </gazebo>
 </robot>

File: src/my_robot_description/urdf/my_robot.urdf.xacro (robot description, xacro)
@@ -149,4 +149,5 @@
      \_____/_/    \_\_____/   |_|  |______|_|  \_\     \/  \/   |_|  |_|______|______|______|
     -->
+    <!-- Caster wheel link -->
     <link name="caster_wheel_link">
         <visual>
@@ -163,5 +164,12 @@
             <origin xyz="0 0 0" rpy="0 0 0" />
         </collision>
-        <xacro:sphere_inertia m="0.5" r="${wheel_radius / 2.0}" o_xyz="0 0 0" o_rpy="0 0 0" />
+        <inertial>
+            <origin xyz="0 0 0" rpy="0 0 0" />
+            <mass value="0.5" />
+            <inertia
+                ixx="0.001" ixy="0.0" ixz="0.0"
+                iyy="0.001" iyz="0.0"
+                izz="0.001" />
+        </inertial>
     </link>
     <joint name="base_caster_wheel_joint" type="fixed">
@@ -170,3 +178,53 @@
         <origin xyz="${base_length / 3.0} 0 -0.05" rpy="0 0 0" />
     </joint>
+    <!-- ==========================
+         FPV CAMERA FOR EMILIOBOT
+         ========================== -->
+    <link name="camera_link">
+        <visual>
+            <geometry>
+                <box size="0.05 0.05 0.05" />
+            </geometry>
+            <origin xyz="0 0 0" rpy="0 0 0" />
+            <material name="black" />
+        </visual>
+        <collision>
+            <geometry>
+                <box size="0.05 0.05 0.05" />
+            </geometry>
+            <origin xyz="0 0 0" rpy="0 0 0" />
+        </collision>
+        <inertial>
+            <origin xyz="0 0 0" rpy="0 0 0" />
+            <mass value="0.1" />
+            <inertia
+                ixx="0.001" ixy="0.0" ixz="0.0"
+                iyy="0.001" iyz="0.0"
+                izz="0.001" />
+        </inertial>
+    </link>
+    <joint name="camera_joint" type="fixed">
+        <parent link="base_link" />
+        <child link="camera_link" />
+        <origin xyz="0 0 ${base_height + 0.1}" rpy="0 0 0" />
+    </joint>
+    <gazebo reference="camera_link">
+        <sensor name="front_camera" type="camera">
+            <always_on>1</always_on>
+            <update_rate>30</update_rate>
+            <visualize>true</visualize>
+            <camera>
+                <horizontal_fov>1.047</horizontal_fov>
+                <image>
+                    <width>640</width>
+                    <height>480</height>
+                    <format>R8G8B8</format>
+                </image>
+                <clip>
+                    <near>0.1</near>
+                    <far>100.0</far>
+                </clip>
+            </camera>
+        </sensor>
+    </gazebo>
 </robot>
